Commit message: Webots: LiDAR frontal 5 cm mais alto e caixotes da arena no piso
O front_lidar sobe de z = -0,15 para -0,10 em relação ao base_link no
agrobot.proto e no URDF: o plano do scan fica a ~13 cm do chão. Na
plantação, os pontos do scan no chão das entrelinhas caem de
651/429/258/447/676 para 80/69/0/50/117 por percurso, e o Nav2 chega a
20 de 20 objetivos (antes 18 de 23).

Os caixotes da arena estavam 5 cm enterrados no piso. A 13 cm, um quarto
dos raios passava pelos vãos das paredes deles; com os caixotes em cima
do piso, o LiDAR os vê como antes. Nav2 na arena: 10 de 10, igual ao
LiDAR antigo.

README e manual com as medições, a altura nova e o estado do
goal_navigator, do EKF e do SLAM no Webots.

Co-Authored-By: Claude Opus 5.5 (1M context) <noreply@anthropic.com>
Claude-Session: https://claude.ai/code/session_01ETUT5vzcmcKbLjihDmyHfJ

File: agrobot_description/urdf/agrobot.urdf (robot description, URDF)
Before this commit: robot agrobot, 10 links, 9 joints
Joints:
- joint front_lidar_joint: origin xyz=0.65 0 -0.15 rpy=0 0 0 -> xyz=0.65 0 -0.10 rpy=0 0 0

Commit message: Webots: RTAB-Map (VSLAM) no launch com câmera RGB-D simulada (vslam:=true)
- agrobot.proto: Camera vslam_color + RangeFinder vslam_depth na mesma pose
  (0,45; 0; 0,38), 15° para baixo, 424 x 240, 87°, 0,5 a 6 m.
- agrobot.urdf: vslam_camera_link e vslam_camera_optical_frame; propriedade
  enableVslamCamera do plugin.
- AgrobotDriver: publica cor, profundidade e camera_info com o mesmo
  carimbo do /scan, a cada 3 passos, só com enableVslamCamera.
- config/rtabmap.yaml: rgbd_sync + rtabmap, odometria pelo TF do EKF,
  registro só visual, grade pelo LiDAR.
- simulation.launch.py: argumentos vslam (exige ekf), vslam_db e
  rtabmap_viz; Nav2 em map com vslam; modo combinado com o slam_toolbox
  sem TF (frame slam_map).
- rviz/nav_vslam.rviz; package.xml com rtabmap_ros.
- README e claude/manual.md com as medições.

Co-Authored-By: Claude Opus 5.5 (1M context) <noreply@anthropic.com>
Claude-Session: https://claude.ai/code/session_01MwmbCFwQWFyqUk1cfV32YM

File: agrobot_description/urdf/agrobot.urdf (robot description, URDF)
Before this commit: robot agrobot, 10 links, 9 joints
Links:
- added link vslam_camera_link
- added link vslam_camera_optical_frame
Joints:
- added joint vslam_camera_joint: type fixed, parent base_link, child vslam_camera_link, origin xyz=0.45 0 0.38 rpy=0 0.2618 0
- added joint vslam_camera_optical_joint: type fixed, parent vslam_camera_link, child vslam_camera_optical_frame, origin xyz=0 0 0 rpy=-1.5708 0 -1.5708
